File: 1.Hardware/RevB-KiCad/Naive/ExtendBoard/ExtendBoard.kicad_sch (KiCad schematic)
At the start: 11 parts, among them CON1 FH12-8S-0.5SH(55), Q1 AO3400A, U1 AL5802

Commit message: Resolve Naive display landing and fabrication rules; add bring-up tools
Parts:
- LCD1: DesignNote P133H002 electrically compatible candidate only; legacy FPC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 -> P133H002 electrically compatible candidate; 5.5x0.5mm F-sid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
Changed lines of the file:
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@@
 			)
 		)
-		(property "DesignNote" "P133H002 electrically compatible candidate only; legacy FPC solder-pad geometry retained. Fold around 1.071mm PCB and enclosure fit unverified; see MECHANICAL-REVIEW.md. External backlight current limiting required."
+		(property "DesignNote" "P133H002 electrically compatible candidate; 5.5x0.5mm F-side solder landing strips at0.7mm pitch provide axial contact-location allowance. FPC is manually soldered AFTER PCBA reflow; no F.Paste apertures. Align all12pins laterally. Permitted bend radius, contact-face orientation and case assembly still require supplier/sample approval; see interface drawing."
 			(at 205.74 87.63 0)
 			(hide yes)

Commit message: Use compatible small-quantity parts in Naive RevB
Parts:
- C4: DesignNote Local 5V bypass, 10V X7R -> Local 5V bypass; 1uF +/-10%, 25V X7R, 0603. Shared MPN with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; MPN GRM188R71A105KA61D -> GRM188R71E105KA12D
Changed lines of the file:
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@@
 			)
 		)
-		(property "Datasheet" ""
+		(property "Datasheet" "https://ds.murata.com/simserve/characteristics?ReqType=TechPDF&partnumber=GRM188R71E105KA12&techpdfname=technical_pdf_Capacitor01&lang=en"
 			(at 377.19 190.5 0)
 			(hide yes)
@@
 			)
 		)
-		(property "MPN" "GRM188R71A105KA61D"
+		(property "MPN" "GRM188R71E105KA12D"
 			(at 377.19 190.5 0)
 			(hide yes)
@@
 			)
 		)
-		(property "DesignNote" "Local 5V bypass, 10V X7R"
+		(property "DesignNote" "Local 5V bypass; 1uF +/-10%, 25V X7R, 0603. Shared MPN with MainBoard C24."
 			(at 377.19 190.5 0)
 			(hide yes)
