File: 1.Hardware/RevB-KiCad/Naive/MainBoard/MainBoard.kicad_pcb (KiCad board)
At the start: 6 copper layers, 28.5 x 23.5 mm, 58 parts, among them CON1 FH12-8S-0.5SH(55), J1 104031-0811, U1 CP2102, U2 TPS62162DSGR, U3 MPU6050, U4 ESP32_SIP, U5 BH1750FVI-TR, U6 TPS22918DBVR, U7 TPD4E05U06DQAR, U8 SN74AHCT1G125DCKR

Commit message: Use compatible small-quantity parts in Naive RevB
Parts:
- U6: value TPS22918DBVR -> TPS22918DBVT
Changed lines of the file:
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@@
 			)
 		)
-		(property "Value" "TPS22918DBVR"
+		(property "Value" "TPS22918DBVT"
 			(at 0 2.4 0)
 			(layer "F.Fab")
@@
 			)
 		)
-		(property "Datasheet" ""
+		(property "Datasheet" "https://www.ti.com/lit/ds/symlink/tps22918.pdf"
 			(at 0 0 0)
 			(layer "F.Fab")
@@
 			)
 		)
-		(property "MPN" "TPS22918DBVR"
+		(property "MPN" "TPS22918DBVT"
 			(at 0 0 0)
 			(layer "F.Fab")
@@
 			)
 		)
-		(property "DesignNote" "QOD unused; ON RC100k/100nF. Quoted slew characterizedVIN stable beforeON; validatehotplug."
+		(property "DesignNote" "TPS22918 DBV6, 250-piece T&R packaging. QOD unused; ON RC100k/100nF. Quoted slew characterized with VIN stable before ON; validate hot-plug."
 			(at 0 0 0)
 			(layer "F.SilkS")
@@
 			)
 		)
-		(property "Datasheet" ""
+		(property "Datasheet" "https://www.ralec.com/upload/media/product/file/IE-SP-010%20.pdf"
 			(at 0 0 90)
 			(layer "F.Fab")
@@
 			)
 		)
-		(property "MPN" "RC0402FR-07200RL"
+		(property "MPN" "RTT022000FTH"
 			(at 0 0 0)
 			(layer "F.SilkS")
@@
 			)
 		)
-		(property "Datasheet" ""
+		(property "Datasheet" "https://ds.murata.com/simserve/characteristics?ReqType=TechPDF&partnumber=GRM188R71E105KA12&techpdfname=technical_pdf_Capacitor01&lang=en"
 			(at 0 0 0)
 			(layer "F.Fab")
@@
 			)
 		)
-		(property "MPN" "GRM188R71C105KA12D"
+		(property "MPN" "GRM188R71E105KA12D"
 			(at 0 0 0)
 			(layer "F.Fab")
@@
 			)
 		)
-		(property "DesignNote" "BH1750 DVI RC sequencing."
+		(property "DesignNote" "BH1750 DVI RC sequencing; 1uF +/-10%, 25V X7R, 0603. Shared MPN with ExtendBoard C4; manufacturer EC curves are typical."
 			(at 0 0 0)
 			(layer "F.SilkS")
