File: 1.Hardware/RevB-KiCad/Naive/MainBoard/MainBoard.kicad_sch (KiCad schematic)
At the start: 58 parts, among them CON1 FH12-8S-0.5SH(55), J1 104031-0811, U1 CP2102, U2 TPS62162DSGR, U3 MPU6050, U4 ESP32_SIP, U5 BH1750FVI-TR, U6 TPS22918DBVR, U7 TPD4E05U06DQAR, U8 SN74AHCT1G125DCKR

Commit message: Use compatible small-quantity parts in Naive RevB
Parts:
- C24: DesignNote BH1750 DVI RC sequencing. -> BH1750 DVI RC sequencing; 1uF +/-10%, 25V X7R, 0603. Shared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; MPN GRM188R71C105KA12D -> GRM188R71E105KA12D
- R3: MPN RC0402FR-07200RL -> RTT022000FTH
- U6: value TPS22918DBVR -> TPS22918DBVT; DesignNote QOD unused; ON RC100k/100nF. Quoted slew characterizedVIN s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 -> TPS22918 DBV6, 250-piece T&R packaging. QOD unused; ON RC10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; MPN TPS22918DBVR -> TPS22918DBVT
Changed lines of the file:
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@@
 			)
 		)
-		(property "Datasheet" ""
+		(property "Datasheet" "https://www.ralec.com/upload/media/product/file/IE-SP-010%20.pdf"
 			(at 59.69 299.72 0)
 			(hide yes)
@@
 			)
 		)
-		(property "MPN" "RC0402FR-07200RL"
+		(property "MPN" "RTT022000FTH"
 			(at 59.69 299.72 0)
 			(hide yes)
@@
 			)
 		)
-		(property "Value" "TPS22918DBVR"
+		(property "Value" "TPS22918DBVT"
 			(at 251.46 45.72 0)
 			(effects
@@
 			)
 		)
-		(property "Datasheet" ""
+		(property "Datasheet" "https://www.ti.com/lit/ds/symlink/tps22918.pdf"
 			(at 251.46 53.34 0)
 			(hide yes)
@@
 			)
 		)
-		(property "MPN" "TPS22918DBVR"
+		(property "MPN" "TPS22918DBVT"
 			(at 251.46 53.34 0)
 			(hide yes)
@@
 			)
 		)
-		(property "DesignNote" "QOD unused; ON RC100k/100nF. Quoted slew characterizedVIN stable beforeON; validatehotplug."
+		(property "DesignNote" "TPS22918 DBV6, 250-piece T&R packaging. QOD unused; ON RC100k/100nF. Quoted slew characterized with VIN stable before ON; validate hot-plug."
 			(at 251.46 53.34 0)
 			(hide yes)
@@
 			)
 		)
-		(property "Datasheet" ""
+		(property "Datasheet" "https://ds.murata.com/simserve/characteristics?ReqType=TechPDF&partnumber=GRM188R71E105KA12&techpdfname=technical_pdf_Capacitor01&lang=en"
 			(at 538.48 238.76 0)
 			(hide yes)
@@
 			)
 		)
-		(property "MPN" "GRM188R71C105KA12D"
+		(property "MPN" "GRM188R71E105KA12D"
 			(at 538.48 238.76 0)
 			(hide yes)
@@
 			)
 		)
-		(property "DesignNote" "BH1750 DVI RC sequencing."
+		(property "DesignNote" "BH1750 DVI RC sequencing; 1uF +/-10%, 25V X7R, 0603. Shared MPN with ExtendBoard C4; manufacturer EC curves are typical."
 			(at 538.48 238.76 0)
 			(hide yes)
